File: OfficeClock/Hardware/Max7219Clock/Max7219Clock.kicad_pcb (KiCad board)
At the start: 2 copper layers, 80 x 40 mm, 6 parts, among them J1 Conn_01x02_Pin, U1 ESP32-C6-Super-Mini, U2 74HCT367, U3 TEMT6000, U4 Max7219 LED Matrix, U5 USB A Header

Commit message: Updated files and generated final Gerber files for submission
Parts:
- added C1: 0.1uf, Capacitor_THT:C_Disc_D8.0mm_W5.0mm_P5.00mm, F.Cu at (170.5, 126.5)
- added C2: 0.1uf, Capacitor_THT:C_Disc_D8.0mm_W5.0mm_P5.00mm, F.Cu at (113.5, 108.5)
- added C3: 0.1uf, Capacitor_THT:C_Disc_D8.0mm_W5.0mm_P5.00mm, F.Cu at (129.5, 125.5)
- added H1: MountingHole, MountingHole:MountingHole_2.2mm_M2, F.Cu at (102.5, 102.5)
- added H2: MountingHole, MountingHole:MountingHole_2.2mm_M2, F.Cu at (177.5, 102.5)
- added H3: MountingHole, MountingHole:MountingHole_2.2mm_M2, F.Cu at (102.5, 137.5)
- added H4: MountingHole, MountingHole:MountingHole_2.2mm_M2, F.Cu at (177.5, 137.5)
- moved J1 12.0 mm to (130.0, 106.5)
Connections:
- J1 pad 1: Net-(J1-Pin_1) -> GND
- J1 pad 2: GND -> Net-(J1-Pin_2)
- U1 pad 14: Net-(J1-Pin_1) -> Net-(J1-Pin_2)
- U2 pad 4: Net-(U1-IO3) -> Net-(U1-IO7)
- U2 pad 6: Net-(U1-IO7) -> Net-(U1-IO3)
Routing:
- net GND: track 159.2 -> 0.00 mm
- net VCC: track 99.1 -> 0.00 mm
- net Net-(J1-Pin_2): track 0.00 -> 26.3 mm
- net Net-(J1-Pin_1): track 25.5 -> 0.00 mm
- net Net-(U1-IO3): track 24.0 -> 21.9 mm
- added copper zone on B.Cu, net GND
- added copper zone on F.Cu, net VCC
